File: ESL_EMITTER.sch (EAGLE design)
At the start: 22 parts, among them IC1 78L05, T1 2N2222, U1 ATTINY85-P

Commit message: feat(labels): add labels & some fix
Other:
- moved on the sheet: C1, C2, C3, C4, C5, C6, D1, D2, GND, IC1, IN, Q1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

Commit message: fix: capacitor&bom : last release
Parts:
- C3, C4: value 10nF -> 22p
- C6: value 10nF -> 3.3nF
- Q1: value (none) -> 10MHz
Changed lines of the file:
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@@
 <part name="V3" library="supply0" deviceset="VBAT" device=""/>
 <part name="U1" library="_hhn_attiny25_45_85" deviceset="ATTINY85*" device="P" technology="-"/>
-<part name="Q1" library="adafruit" deviceset="CRYSTAL" device="HC49U-H"/>
-<part name="C3" library="SparkFun-Capacitors" deviceset="10NF" device="-PTH-10MM-10000V-1-%" value="10nF"/>
-<part name="C4" library="SparkFun-Capacitors" deviceset="10NF" device="-PTH-10MM-10000V-1-%" value="10nF"/>
+<part name="Q1" library="adafruit" deviceset="CRYSTAL" device="HC49U-H" value="10MHz"/>
+<part name="C3" library="SparkFun-Capacitors" deviceset="10NF" device="-PTH-10MM-10000V-1-%" value="22p"/>
+<part name="C4" library="SparkFun-Capacitors" deviceset="10NF" device="-PTH-10MM-10000V-1-%" value="22p"/>
 <part name="GND4" library="supply" deviceset="GND" device=""/>
 <part name="R1" library="resistor" deviceset="R-EU_" device="0207/7" value="3.3k"/>
@@
 <part name="C5" library="SparkFun" deviceset="CAP_POL" device="PTH2" value="100uF"/>
 <part name="T1" library="adafruit" deviceset="2N2222" device=""/>
-<part name="C6" library="SparkFun-Capacitors" deviceset="10NF" device="-PTH-10MM-10000V-1-%" value="10nF"/>
+<part name="C6" library="SparkFun-Capacitors" deviceset="10NF" device="-PTH-10MM-10000V-1-%" value="3.3nF"/>
 <part name="GND6" library="supply" deviceset="GND" device=""/>
 <part name="R5" library="resistor" deviceset="R-EU_" device="0207/7" value="220r"/>
@@
 <instance part="C3" gate="G$1" x="167.64" y="99.06" smashed="yes">
 <attribute name="NAME" x="169.164" y="101.981" size="1.778" layer="95" font="vector"/>
-<attribute name="VALUE" x="159.004" y="96.901" size="1.778" layer="96" font="vector"/>
+<attribute name="VALUE" x="161.544" y="96.901" size="1.778" layer="96" font="vector"/>
 </instance>
 <instance part="C4" gate="G$1" x="172.72" y="99.06" smashed="yes">
